Commit message: Adding Localiaztion and Control
- Added Kalman Filter example file
- Added PD Controller
- fixed slippage of wheels (has to be better fixed later, for now it is ok)

File: simulation_environment/models/diff_drive/diff_drive.xacro (robot description, xacro)
@@ -63,8 +63,8 @@
         <friction>
           <ode>
-            <mu>1000</mu>
-            <mu2>1000</mu2>
-            <slip1>1.0</slip1>
-            <slip2>1.0</slip2>
+            <mu>1.0</mu>
+            <mu2>1.0</mu2>
+            <slip1>0.0</slip1>
+            <slip2>0.0</slip2>
           </ode>
         </friction>
@@ -93,8 +93,8 @@
         <friction>
           <ode>
-            <mu>1000</mu>
-            <mu2>1000</mu2>
-            <slip1>1.0</slip1>
-            <slip2>1.0</slip2>
+            <mu>1.0</mu>
+            <mu2>1.0</mu2>
+            <slip1>0.0</slip1>
+            <slip2>0.0</slip2>
           </ode>
         </friction>

File: simulation_environment/models/diff_drive/parameter.xacro (robot description, xacro)
@@ -1,4 +1,7 @@
 <?xml version="1.0"?>
 <robot xmlns:xacro="http://www.ros.org/wiki/xacro">
+  <!-- Load config file, TODO: Add more parameter -->
+  <xacro:property name="package" value="$(find simulation_environment)"/>
+  <xacro:property name="properties" value="${load_yaml(package + '/config/config.yaml')}"/>
   <!-- Define parameter for the differential drive robot -->
   <!-- Parameter for the chassis, size [m] and mass [kg] -->
@@ -8,9 +11,12 @@
   <xacro:property name="m_chassis" value="5.0" />
   <!-- Parameter for the wheels, radius [m], height [m], mass [kg], torque [Nm], wheelbase [m] -->
-  <xacro:property name="r_wheel" value="0.1075" />
+  <xacro:property name="r_wheel" value="${properties['wheel_radius']}"/>
   <xacro:property name="h_wheel" value="0.03" />
-  <xacro:property name="m_wheel" value="0.5" />
+  <xacro:property name="m_wheel" value="10.0" />
   <xacro:property name="torque_wheel" value="100" />
-  <xacro:property name="L_wheel" value="0.1788" />
+  <xacro:property name="L_wheel" value="${properties['axis_distance']}" />
+  <!-- Noise parameter for the differential drive -->
+  <xacro:property name="noise_vel" value="${properties['noise_vel']}" />
+  <xacro:property name="noise_odom" value="${properties['noise_odom']}" />
   <!-- Parameters for the Hukoyu Laser -->
   <xacro:property name="x_hokuyo" value="0.1" />

Commit message: Update Sim Environment
- Added Odom link as reference for the odometry center
- Added frames to /imu and /odom topics

File: simulation_environment/models/diff_drive/diff_drive.xacro (robot description, xacro)
@@ -53,4 +53,24 @@
     </visual>
   </link>
+  <!-- Add an odom link -->
+  <link name="odom_link" >
+	<collision>
+      <origin xyz="0 0 0" rpy="0 0 0"/>
+      <geometry>
+		<box size="1e-6 1e-6 1e-6"/>
+      </geometry>
+    </collision>
+    <inertial>
+      <mass value="1e-5" />
+      <origin xyz="0 0 0" rpy="0 0 0"/>
+      <inertia ixx="1e-6" ixy="0" ixz="0" iyy="1e-6" iyz="0" izz="1e-6" />
+    </inertial>
+  </link>
+  <joint name="odom_joint" type="fixed">
+    <axis xyz="0 1 0" />
+    <origin xyz="${-x_chassis/4} 0 0" rpy="0 0 0"/>
+    <parent link="base_link"/>
+    <child link="odom_link"/>
+  </joint>
   <!-- Add the wheels for the robot -->
   <link name="left_wheel">
@@ -116,7 +136,7 @@
   <!-- Set joints for the wheels which can be controlled over ROS -->
   <joint type="continuous" name="left_wheel_hinge">
-    <origin xyz="${-x_chassis/4} ${y_chassis/2+h_wheel/2} ${r_wheel/2-z_chassis/2}" rpy="0 0 0"/>
+    <origin xyz="0 ${y_chassis/2+h_wheel/2} ${r_wheel/2-z_chassis/2}" rpy="0 0 0"/>
     <child link="left_wheel"/>
-    <parent link="base_link"/>
+    <parent link="odom_link"/>
     <axis xyz="0 1 0" rpy="0 0 0"/>
     <limit effort="100" velocity="100"/>
@@ -124,7 +144,7 @@
   </joint>
   <joint type="continuous" name="right_wheel_hinge">
-    <origin xyz="${-x_chassis/4} ${-y_chassis/2-h_wheel/2} ${r_wheel/2-z_chassis/2}" rpy="0 0 0"/>
+    <origin xyz="0 ${-y_chassis/2-h_wheel/2} ${r_wheel/2-z_chassis/2}" rpy="0 0 0"/>
     <child link="right_wheel"/>
-    <parent link="base_link"/>
+    <parent link="odom_link"/>
     <axis xyz="0 1 0" rpy="0 0 0"/>
     <limit effort="100" velocity="100"/>

File: simulation_environment/models/diff_drive/parameter.xacro (robot description, xacro)
@@ -9,10 +9,10 @@
   <xacro:property name="y_chassis" value="0.3" />
   <xacro:property name="z_chassis" value="0.15" />
-  <xacro:property name="m_chassis" value="5.0" />
+  <xacro:property name="m_chassis" value="10.0" />
   <!-- Parameter for the wheels, radius [m], height [m], mass [kg], torque [Nm], wheelbase [m] -->
   <xacro:property name="r_wheel" value="${properties['wheel_radius']}"/>
   <xacro:property name="h_wheel" value="0.03" />
-  <xacro:property name="m_wheel" value="10.0" />
-  <xacro:property name="torque_wheel" value="100" />
+  <xacro:property name="m_wheel" value="3.0" />
+  <xacro:property name="torque_wheel" value="10" />
   <xacro:property name="L_wheel" value="${properties['axis_distance']}" />
   <!-- Noise parameter for the differential drive -->
@@ -23,3 +23,7 @@
   <xacro:property name="y_hokuyo" value="0.1" />
   <xacro:property name="z_hokuyo" value="0.1" />
+    <!-- Parameters for the IMU -->
+  <xacro:property name="x_imu" value="0.01" />
+  <xacro:property name="y_imu" value="0.01" />
+  <xacro:property name="z_imu" value="0.01" />
 </robot>

Commit message: Update Tutorial for Rescue Robotic Exercises

File: simulation_environment/models/diff_drive/diff_drive.xacro (robot description, xacro)
@@ -7,5 +7,5 @@
   <xacro:include filename="$(find simulation_environment)/models/diff_drive/macros.xacro"      />
   <xacro:include filename="$(find simulation_environment)/models/diff_drive/parameter.xacro"   />
-  <!-- Define the chassis of the differential drive robot -->
+  <!-- Define the chassis of the differential drive robot, which is our base -->
   <link name='base_link'>
     <pose>0 0 0 0 0 0</pose>
@@ -53,24 +53,4 @@
     </visual>
   </link>
-  <!-- Add an odom link -->
-  <link name="odom_link" >
-	<collision>
-      <origin xyz="0 0 0" rpy="0 0 0"/>
-      <geometry>
-		<box size="1e-6 1e-6 1e-6"/>
-      </geometry>
-    </collision>
-    <inertial>
-      <mass value="1e-5" />
-      <origin xyz="0 0 0" rpy="0 0 0"/>
-      <inertia ixx="1e-6" ixy="0" ixz="0" iyy="1e-6" iyz="0" izz="1e-6" />
-    </inertial>
-  </link>
-  <joint name="odom_joint" type="fixed">
-    <axis xyz="0 1 0" />
-    <origin xyz="${-x_chassis/4} 0 0" rpy="0 0 0"/>
-    <parent link="base_link"/>
-    <child link="odom_link"/>
-  </joint>
   <!-- Add the wheels for the robot -->
   <link name="left_wheel">
@@ -136,7 +116,7 @@
   <!-- Set joints for the wheels which can be controlled over ROS -->
   <joint type="continuous" name="left_wheel_hinge">
-    <origin xyz="0 ${y_chassis/2+h_wheel/2} ${r_wheel/2-z_chassis/2}" rpy="0 0 0"/>
+    <origin xyz="${-x_chassis/4} ${y_chassis/2+h_wheel/2} ${r_wheel/2-z_chassis/2}" rpy="0 0 0"/>
     <child link="left_wheel"/>
-    <parent link="odom_link"/>
+    <parent link="base_link"/>
     <axis xyz="0 1 0" rpy="0 0 0"/>
     <limit effort="100" velocity="100"/>
@@ -144,7 +124,7 @@
   </joint>
   <joint type="continuous" name="right_wheel_hinge">
-    <origin xyz="0 ${-y_chassis/2-h_wheel/2} ${r_wheel/2-z_chassis/2}" rpy="0 0 0"/>
+    <origin xyz="${-x_chassis/4} ${-y_chassis/2-h_wheel/2} ${r_wheel/2-z_chassis/2}" rpy="0 0 0"/>
     <child link="right_wheel"/>
-    <parent link="odom_link"/>
+    <parent link="base_link"/>
     <axis xyz="0 1 0" rpy="0 0 0"/>
     <limit effort="100" velocity="100"/>

Commit message: Update Human Model and add camera

File: simulation_environment/models/diff_drive/diff_drive.xacro (robot description, xacro)
@@ -132,5 +132,5 @@
   </joint>
   <!-- Add a Hokuyo Laser -->
-  <link name="laser">
+  <link name="laser_link">
     <collision>
       <origin xyz="0 0 0" rpy="0 0 0"/>
@@ -156,5 +156,32 @@
     <origin xyz="0 0 ${z_chassis/2 + z_hokuyo/2}" rpy="0 0 0"/>
     <parent link="base_link"/>
-    <child link="laser"/>
+    <child link="laser_link"/>
+  </joint>
+  <!-- Add the camera link -->
+  <link name="camera_link">
+    <collision>
+      <origin xyz="0 0 0" rpy="0 0 0"/>
+      <geometry>
+    <box size="${camera_size} ${camera_size} ${camera_size}"/>
+      </geometry>
+    </collision>
+    <visual>
+      <origin xyz="0 0 0" rpy="0 0 0"/>
+      <geometry>
+    <box size="${camera_size} ${camera_size} ${camera_size}"/>
+      </geometry>
+      <material name="red"/>
+    </visual>
+    <inertial>
+      <mass value="1e-5" />
+      <origin xyz="0 0 0" rpy="0 0 0"/>
+      <inertia ixx="1e-6" ixy="0" ixz="0" iyy="1e-6" iyz="0" izz="1e-6" />
+    </inertial>
+  </link>
+  <joint name="camera_joint" type="fixed">
+    <axis xyz="0 1 0" />
+    <origin xyz="0 0 ${z_hokuyo/2 + camera_size/2}" rpy="0 0 0"/>
+    <parent link="laser_link"/>
+    <child link="camera_link"/>
   </joint>
  </robot>

File: simulation_environment/models/diff_drive/parameter.xacro (robot description, xacro)
@@ -27,3 +27,5 @@
   <xacro:property name="y_imu" value="0.01" />
   <xacro:property name="z_imu" value="0.01" />
+  <!-- Camera -->
+  <xacro:property name="camera_size" value="0.05" />
 </robot>

Commit message: Fixed LaserScan Frame Problem and Odom KDF Problem

File: simulation_environment/models/diff_drive/diff_drive.xacro (robot description, xacro)
@@ -7,6 +7,14 @@
   <xacro:include filename="$(find simulation_environment)/models/diff_drive/macros.xacro"      />
   <xacro:include filename="$(find simulation_environment)/models/diff_drive/parameter.xacro"   />
+ <!-- Create a dummy link as base link -->
+  <link name='base_link'>
+    <pose>0 0 0 0 0 0</pose>
+  </link>
+  <joint type="fixed" name="base_link_to_chassis">
+    <child link="chassis_link"/>
+    <parent link="base_link"/>
+  </joint>
   <!-- Define the chassis of the differential drive robot, which is our base -->
-  <link name='base_link'>
+  <link name='chassis_link'>
     <pose>0 0 0 0 0 0</pose>
     <!-- Define inertial system for the chassis -->
